Commit message: added gripper name and fixed typos

File: gripper_description/urdf/gripper.gazebo.xacro (robot description, xacro)
@@ -1,13 +1,13 @@
 <?xml version="1.0"?>
 <robot xmlns:xacro="http://www.ros.org/wiki/xacro">
-    <xacro:macro name="gripper_gazebo" params="robot_name">
+    <xacro:macro name="gripper_gazebo" params="gripper_name">
         <!-- ros_control-plugin -->
         <gazebo>
             <plugin name="gazebo_ros_control" filename="libgazebo_ros_control.so">
-                <robotNamespace>/${robot_name}</robotNamespace>
+                <robotNamespace>/${gripper_name}</robotNamespace>
             </plugin>
         </gazebo>
         <!-- link 0 -->
-        <gazebo reference="link_0">
+        <gazebo reference="${gripper_name}_link_0">
             <mu1>0.2</mu1>
             <mu2>0.2</mu2>
@@ -15,5 +15,5 @@
         </gazebo>
         <!-- link 1 -->
-        <gazebo reference="link_1">
+        <gazebo reference="${gripper_name}_link_1">
             <mu1>0.2</mu1>
             <mu2>0.2</mu2>
@@ -21,5 +21,5 @@
         </gazebo>
         <!-- link 2 -->
-        <gazebo reference="link_2">
+        <gazebo reference="${gripper_name}_link_2">
             <mu1>0.2</mu1>
             <mu2>0.2</mu2>
@@ -27,5 +27,5 @@
         </gazebo>
         <!-- link 3 -->
-        <gazebo reference="link_3">
+        <gazebo reference="${gripper_name}_link_3">
             <mu1>0.2</mu1>
             <mu2>0.2</mu2>
@@ -33,5 +33,5 @@
         </gazebo>
         <!-- link 4 -->
-        <gazebo reference="link_4">
+        <gazebo reference="${gripper_name}_link_4">
             <mu1>0.2</mu1>
             <mu2>0.2</mu2>

File: gripper_description/urdf/gripper.transmission.xacro (robot description, xacro)
@@ -1,13 +1,13 @@
 <?xml version="1.0"?>
 <robot xmlns:xacro="http://www.ros.org/wiki/xacro">
-    <xacro:macro name="gripper_transmission" params="hardware_interface robot_name">
+    <xacro:macro name="gripper_transmission" params="hardware_interface gripper_name">
         <!-- joint 1 -->
-        <transmission name="tran_1">
-            <robotNamespace>/${robot_name}</robotNamespace>
+        <transmission name="${gripper_name}_tran_1">
+            <robotNamespace>/${gripper_name}</robotNamespace>
             <type>transmission_interface/SimpleTransmission</type>
-            <joint name="joint_1">
+            <joint name="${gripper_name}_joint_1">
                 <hardwareInterface>hardware_interface/${hardware_interface}</hardwareInterface>
             </joint>
-            <actuator name="motor_1">
+            <actuator name="${gripper_name}_motor_1">
                 <hardwareInterface>hardware_interface/${hardware_interface}</hardwareInterface>
                 <mechanicalReduction>1</mechanicalReduction>
@@ -15,11 +15,11 @@
         </transmission>
         <!-- joint 2 -->
-        <transmission name="tran_2">
-            <robotNamespace>/${robot_name}</robotNamespace>
+        <transmission name="${gripper_name}_tran_2">
+            <robotNamespace>/${gripper_name}</robotNamespace>
             <type>transmission_interface/SimpleTransmission</type>
-            <joint name="joint_2">
+            <joint name="${gripper_name}_joint_2">
                 <hardwareInterface>hardware_interface/${hardware_interface}</hardwareInterface>
             </joint>
-            <actuator name="motor_2">
+            <actuator name="${gripper_name}_motor_2">
                 <hardwareInterface>hardware_interface/${hardware_interface}</hardwareInterface>
                 <mechanicalReduction>1</mechanicalReduction>
@@ -27,11 +27,11 @@
         </transmission>
         <!-- joint 3 -->
-        <transmission name="tran_3">
-            <robotNamespace>/${robot_name}</robotNamespace>
+        <transmission name="${gripper_name}_tran_3">
+            <robotNamespace>/${gripper_name}</robotNamespace>
             <type>transmission_interface/SimpleTransmission</type>
-            <joint name="joint_3">
+            <joint name="${gripper_name}_joint_3">
                 <hardwareInterface>hardware_interface/${hardware_interface}</hardwareInterface>
             </joint>
-            <actuator name="motor_3">
+            <actuator name="${gripper_name}_motor_3">
                 <hardwareInterface>hardware_interface/${hardware_interface}</hardwareInterface>
                 <mechanicalReduction>1</mechanicalReduction>
@@ -39,11 +39,11 @@
         </transmission>
         <!-- joint 4 -->
-        <transmission name="tran_4">
-            <robotNamespace>/${robot_name}</robotNamespace>
+        <transmission name="${gripper_name}_tran_4">
+            <robotNamespace>/${gripper_name}</robotNamespace>
             <type>transmission_interface/SimpleTransmission</type>
-                <joint name="joint_4">
+                <joint name="${gripper_name}_joint_4">
             <hardwareInterface>hardware_interface/${hardware_interface}</hardwareInterface>
             </joint>
-            <actuator name="motor_4">
+            <actuator name="${gripper_name}_motor_4">
                 <hardwareInterface>hardware_interface/${hardware_interface}</hardwareInterface>
                 <mechanicalReduction>1</mechanicalReduction>

File: gripper_description/urdf/gripper.xacro (robot description, xacro)
@@ -1,153 +1,154 @@
 <?xml version="1.0" ?>
 <robot xmlns:xacro="http://www.ros.org/wiki/xacro">
-    <xacro:macro name="gripper" params="hardware_interface parent robot_name">
-    <!-- include gazebo specifications -->
-    <xacro:include filename="$(find gripper_description)/urdf/gripper.gazebo.xacro"/>
-    <!-- include transmission for ros_control -->
-    <xacro:include filename="$(find gripper_description)/urdf/gripper.transmission.xacro"/>
-    <!--joint between {parent} and link_0-->
-    <joint name="${parent}_${robot_name}_joint" type="fixed">
-        <parent link="${parent}"/>
-        <child link="link_0"/>
-    </joint>
-    <link name="link_0">
-        <inertial>
-        <origin rpy="0 0 0" xyz="-6.432910810921765e-05 -0.01226896702938846 0.04229819263832419"/>
-        <mass value="3.001662804726904"/>
-        <inertia ixx="0.013056" ixy="1e-05" ixz="4e-06" iyy="0.002133" iyz="0.000838" izz="0.012592"/>
-        </inertial>
-        <visual>
-        <origin rpy="0 0 0" xyz="0 0 0"/>
-        <geometry>
-            <mesh filename="package://gripper_description/meshes/visual/link_0.stl"/>
-        </geometry>
-        <material name="silver">
-            <color rgba="1 0 0 1"/>
-        </material>
-        </visual>
-        <collision>
-        <origin rpy="0 0 0" xyz="0 0 0"/>
-        <geometry>
-            <mesh filename="package://gripper_description/meshes/collision/link_0.stl"/>
-        </geometry>
-        </collision>
-    </link>
-    <joint name="joint_1" type="continuous">
-        <origin rpy="0 0 0" xyz="0.0 -0.417886 0.064767"/>
-        <parent link="link_0"/>
-        <child link="link_1"/>
-        <axis xyz="-0.0 -0.01 8.3e-05"/>
-    </joint>
-    <link name="link_1">
-        <inertial>
-        <origin rpy="0 0 0" xyz="7.83131813835923e-13 -0.00327664993849075 2.7009925125554002e-05"/>
-        <mass value="0.0026081265321506496"/>
-        <inertia ixx="0.0" ixy="-0.0" ixz="0.0" iyy="0.0" iyz="0.0" izz="0.0"/>
-        </inertial>
-        <visual>
-        <origin rpy="0 0 0" xyz="0.0 0.417886 -0.064767"/>
-        <geometry>
-            <mesh filename="package://gripper_description/meshes/visual/link_1.stl"/>
-        </geometry>
-        <material name="silver">
-            <color rgba="1 0 0 1"/>
-        </material>
-        </visual>
-        <collision>
-        <origin rpy="0 0 0" xyz="0.0 0.417886 -0.064767"/>
-        <geometry>
-            <mesh filename="package://gripper_description/meshes/collision/link_1.stl"/>
-        </geometry>
-        </collision>
-    </link>
-    <joint name="joint_2" type="revolute">
-        <origin rpy="0 0 0" xyz="0.004011 -0.0091 7.5e-05"/>
-        <parent link="link_1"/>
-        <child link="link_2"/>
-        <axis xyz="0.01 0.0 0.0"/>
-        <limit effort="100" lower="-1.570796" upper="1.570796" velocity="100"/>
-    </joint>
-    <link name="link_2">
-        <inertial>
-        <origin rpy="0 0 0" xyz="-0.004011372054136788 -0.0036950459896274435 -1.8961420446314547e-05"/>
-        <mass value="0.002076310514419514"/>
-        <inertia ixx="0.0" ixy="-0.0" ixz="-0.0" iyy="0.0" iyz="0.0" izz="0.0"/>
-        </inertial>
-        <visual>
-        <origin rpy="0 0 0" xyz="-0.004011 0.426986 -0.064842"/>
-        <geometry>
-            <mesh filename="package://gripper_description/meshes/visual/link_2.stl"/>
-        </geometry>
-        <material name="silver">
-            <color rgba="1 0 0 1"/>
-        </material>
-        </visual>
-        <collision>
-        <origin rpy="0 0 0" xyz="-0.004011 0.426986 -0.064842"/>
-        <geometry>
-            <mesh filename="package://gripper_description/meshes/collision/link_2.stl"/>
-        </geometry>
-        </collision>
-    </link>
-    <joint name="joint_3" type="revolute">
-        <origin rpy="0 0 0" xyz="-0.003995 -0.008884 0.001974"/>
-        <parent link="link_2"/>
-        <child link="link_3"/>
-        <axis xyz="-8.3e-05 -8.3e-05 -0.009999"/>
-        <limit effort="100" lower="-1.047198" upper="2.094395" velocity="100"/>
-    </joint>
-    <link name="link_3">
-        <inertial>
-        <origin rpy="0 0 0" xyz="0.004525594967446788 -0.006690181259015049 -0.0015230283617313073"/>
-        <mass value="0.000770269058655591"/>
-        <inertia ixx="0.0" ixy="0.0" ixz="0.0" iyy="0.0" iyz="-0.0" izz="0.0"/>
-        </inertial>
-        <visual>
-        <origin rpy="0 0 0" xyz="-1.6e-05 0.43587 -0.066816"/>
-        <geometry>
-            <mesh filename="package://gripper_description/meshes/visual/link_3.stl"/>
-        </geometry>
-        <material name="silver">
-            <color rgba="1 0 0 1"/>
-        </material>
-        </visual>
-        <collision>
-        <origin rpy="0 0 0" xyz="-1.6e-05 0.43587 -0.066816"/>
-        <geometry>
-            <mesh filename="package://gripper_description/meshes/collision/link_3.stl"/>
-        </geometry>
-        </collision>
-    </link>
-    <joint name="joint_4" type="revolute">
-        <origin rpy="0 0 0" xyz="-0.004028 -0.008916 -0.001926"/>
-        <parent link="link_2"/>
-        <child link="link_4"/>
-        <axis xyz="8.3e-05 8.3e-05 0.009999"/>
-        <limit effort="100" lower="-1.047198" upper="2.094395" velocity="100"/>
-    </joint>
-    <link name="link_4">
-        <inertial>
-        <origin rpy="0 0 0" xyz="-0.004531793856768577 -0.006670291152332475 0.00163086900587045"/>
-        <mass value="0.0007630222199738701"/>
-        <inertia ixx="0.0" ixy="-0.0" ixz="0.0" iyy="0.0" iyz="0.0" izz="0.0"/>
-        </inertial>
-        <visual>
-        <origin rpy="0 0 0" xyz="1.7e-05 0.435902 -0.062916"/>
-        <geometry>
-            <mesh filename="package://gripper_description/meshes/visual/link_4.stl"/>
-        </geometry>
-        <material name="silver">
-            <color rgba="1 0 0 1"/>
-        </material>
-        </visual>
-        <collision>
-        <origin rpy="0 0 0" xyz="1.7e-05 0.435902 -0.062916"/>
-        <geometry>
-            <mesh filename="package://gripper_description/meshes/collision/link_4.stl"/>
-        </geometry>
-        </collision>
-    </link>
-    <!-- extensions -->
-    <xacro:gripper_gazebo robot_name="${robot_name}"/>
-    <xacro:gripper_transmission hardware_interface="${hardware_interface}" robot_name="${robot_name}"/>
+    <xacro:macro name="gripper" params="gripper_name hardware_interface parent">
+        <!-- include gazebo specifications -->
+        <xacro:include filename="$(find gripper_description)/urdf/gripper.gazebo.xacro"/>
+        <!-- include transmission for ros_control -->
+        <xacro:include filename="$(find gripper_description)/urdf/gripper.transmission.xacro"/>
+        <!--joint between {parent} and link_0-->
+        <joint name="${parent}_${gripper_name}_joint" type="fixed">
+            <parent link="${parent}"/>
+            <child link="${gripper_name}_link_0"/>
+        </joint>
+        <link name="${gripper_name}_link_0">
+            <inertial>
+                <origin rpy="0 0 0" xyz="-6.432910810921765e-05 -0.01226896702938846 0.04229819263832419"/>
+                <mass value="3.001662804726904"/>
+                <inertia ixx="0.013056" ixy="1e-05" ixz="4e-06" iyy="0.002133" iyz="0.000838" izz="0.012592"/>
+            </inertial>
+            <visual>
+                <origin rpy="0 0 0" xyz="0 0 0"/>
+                <geometry>
+                    <mesh filename="package://gripper_description/meshes/visual/link_0.stl"/>
+                </geometry>
+                <material name="silver">
+                    <color rgba="1 0 0 1"/>
+                </material>
+            </visual>
+            <collision>
+                <origin rpy="0 0 0" xyz="0 0 0"/>
+                <geometry>
+                    <mesh filename="package://gripper_description/meshes/collision/link_0.stl"/>
+                </geometry>
+            </collision>
+        </link>
+        <joint name="${gripper_name}_joint_1" type="continuous">
+            <origin rpy="0 0 0" xyz="0.0 -0.417886 0.064767"/>
+            <parent link="${gripper_name}_link_0"/>
+            <child link="${gripper_name}_link_1"/>
+            <axis xyz="-0.0 -0.01 8.3e-05"/>
+        </joint>
+        <link name="${gripper_name}_link_1">
+            <inertial>
+                <origin rpy="0 0 0" xyz="7.83131813835923e-13 -0.00327664993849075 2.7009925125554002e-05"/>
+                <mass value="0.0026081265321506496"/>
+                <inertia ixx="0.0" ixy="-0.0" ixz="0.0" iyy="0.0" iyz="0.0" izz="0.0"/>
+            </inertial>
+            <visual>
+                <origin rpy="0 0 0" xyz="0.0 0.417886 -0.064767"/>
+                <geometry>
+                    <mesh filename="package://gripper_description/meshes/visual/link_1.stl"/>
+                </geometry>
+                <material name="silver">
+                    <color rgba="1 0 0 1"/>
+                </material>
+            </visual>
+            <collision>
+                <origin rpy="0 0 0" xyz="0.0 0.417886 -0.064767"/>
+                <geometry>
+                    <mesh filename="package://gripper_description/meshes/collision/link_1.stl"/>
+                </geometry>
+            </collision>
+        </link>
+        <joint name="${gripper_name}_joint_2" type="revolute">
+            <origin rpy="0 0 0" xyz="0.004011 -0.0091 7.5e-05"/>
+            <parent link="${gripper_name}_link_1"/>
+            <child link="${gripper_name}_link_2"/>
+            <axis xyz="0.01 0.0 0.0"/>
+            <limit effort="100" lower="-1.570796" upper="1.570796" velocity="100"/>
+        </joint>
+        <link name="${gripper_name}_link_2">
+            <inertial>
+                <origin rpy="0 0 0" xyz="-0.004011372054136788 -0.0036950459896274435 -1.8961420446314547e-05"/>
+                <mass value="0.002076310514419514"/>
+                <inertia ixx="0.0" ixy="-0.0" ixz="-0.0" iyy="0.0" iyz="0.0" izz="0.0"/>
+            </inertial>
+            <visual>
+                <origin rpy="0 0 0" xyz="-0.004011 0.426986 -0.064842"/>
+                <geometry>
+                    <mesh filename="package://gripper_description/meshes/visual/link_2.stl"/>
+                </geometry>
+                <material name="silver">
+                    <color rgba="1 0 0 1"/>
+                </material>
+            </visual>
+            <collision>
+                <origin rpy="0 0 0" xyz="-0.004011 0.426986 -0.064842"/>
+                <geometry>
+                    <mesh filename="package://gripper_description/meshes/collision/link_2.stl"/>
+                </geometry>
+            </collision>
+        </link>
+        <joint name="${gripper_name}_joint_3" type="revolute">
+            <origin rpy="0 0 0" xyz="-0.003995 -0.008884 0.001974"/>
+            <parent link="${gripper_name}_link_2"/>
+            <child link="${gripper_name}_link_3"/>
+            <axis xyz="-8.3e-05 -8.3e-05 -0.009999"/>
+            <limit effort="100" lower="-1.047198" upper="2.094395" velocity="100"/>
+        </joint>
+        <link name="${gripper_name}_link_3">
+            <inertial>
+                <origin rpy="0 0 0" xyz="0.004525594967446788 -0.006690181259015049 -0.0015230283617313073"/>
+                <mass value="0.000770269058655591"/>
+                <inertia ixx="0.0" ixy="0.0" ixz="0.0" iyy="0.0" iyz="-0.0" izz="0.0"/>
+            </inertial>
+                <visual>
+                <origin rpy="0 0 0" xyz="-1.6e-05 0.43587 -0.066816"/>
+                <geometry>
+                    <mesh filename="package://gripper_description/meshes/visual/link_3.stl"/>
+                </geometry>
+                <material name="silver">
+                    <color rgba="1 0 0 1"/>
+                </material>
+            </visual>
+            <collision>
+                <origin rpy="0 0 0" xyz="-1.6e-05 0.43587 -0.066816"/>
+                <geometry>
+                    <mesh filename="package://gripper_description/meshes/collision/link_3.stl"/>
+                </geometry>
+            </collision>
+        </link>
+        <joint name="${gripper_name}_joint_4" type="revolute">
+            <origin rpy="0 0 0" xyz="-0.004028 -0.008916 -0.001926"/>
+            <parent link="${gripper_name}_link_2"/>
+            <child link="${gripper_name}_link_4"/>
+            <axis xyz="8.3e-05 8.3e-05 0.009999"/>
+            <limit effort="100" lower="-1.047198" upper="2.094395" velocity="100"/>
+        </joint>
+        <link name="${gripper_name}_link_4">
+            <inertial>
+                <origin rpy="0 0 0" xyz="-0.004531793856768577 -0.006670291152332475 0.00163086900587045"/>
+                <mass value="0.0007630222199738701"/>
+                <inertia ixx="0.0" ixy="-0.0" ixz="0.0" iyy="0.0" iyz="0.0" izz="0.0"/>
+            </inertial>
+            <visual>
+                <origin rpy="0 0 0" xyz="1.7e-05 0.435902 -0.062916"/>
+                <geometry>
+                    <mesh filename="package://gripper_description/meshes/visual/link_4.stl"/>
+                </geometry>
+                <material name="silver">
+                    <color rgba="1 0 0 1"/>
+                </material>
+            </visual>
+            <collision>
+                <origin rpy="0 0 0" xyz="1.7e-05 0.435902 -0.062916"/>
+                <geometry>
+                    <mesh filename="package://gripper_description/meshes/collision/link_4.stl"/>
+                </geometry>
+            </collision>
+        </link>
+        <!-- extensions -->
+        <xacro:gripper_gazebo gripper_name="${gripper_name}"/>
+        <xacro:gripper_transmission hardware_interface="${hardware_interface}" gripper_name="${gripper_name}"/>
+    </xacro:macro>
 </robot>
