Commit message: updated joint ee

File: gripper_description/urdf/gripper.xacro (robot description, xacro)
@@ -10,4 +10,5 @@
             <parent link="${parent}"/>
             <child link="${gripper_name}_link_0"/>
+            <origin rpy="0 0 1.57079632679" xyz="0 0 0"/>
         </joint>
         <link name="${gripper_name}_link_0">
@@ -148,4 +149,11 @@
             </collision>
         </link>
+        <joint name="${gripper_name}_joint_ee" type="fixed">
+            <origin rpy="0 0 0" xyz="-0.004028 -0.028766 -0.001926"/>
+            <parent link="${gripper_name}_link_2"/>
+            <child link="${gripper_name}_ee"/>
+        </joint>
+        <link name="${gripper_name}_ee">
+        </link>
         <!-- extensions -->
         <xacro:gripper_gazebo gripper_name="${gripper_name}"/>
