Commit message: removed typo

File: endoscope_description/urdf/endoscope.transmission.xacro (robot description, xacro)
@@ -4,5 +4,5 @@
         <!-- joint 1 -->
         <transmission name="${endoscope_name}_tran_1">
-            <robotNamespace>/${gripper_name}</robotNamespace>
+            <robotNamespace>/${endoscope_name}</robotNamespace>
             <type>transmission_interface/SimpleTransmission</type>
             <joint name="${endoscope_name}_joint_1">

File: endoscope_description/urdf/endoscope.xacro (robot description, xacro)
@@ -1,5 +1,5 @@
 <?xml version="1.0"?>
 <robot xmlns:xacro="http://www.ros.org/wiki/xacro">
-    <xacro:macro name="endoscope" params="endoscope_name parent">
+    <xacro:macro name="endoscope" params="endoscope_name hardware_interface parent">
         <!-- include gazebo specifications -->
         <xacro:include filename="$(find endoscope_description)/urdf/endoscope.gazebo.xacro"/>
@@ -24,6 +24,6 @@
                     <mesh filename="package://endoscope_description/meshes/visual/link_0.stl"/>
                 </geometry>
-                <material name="silver">
-                    <color rgba="1 0 0 1"/>
+                <material name="white">
+                    <color rgba="1.0 1.0 1.0 1.0"/>
                 </material>
             </visual>
@@ -73,5 +73,5 @@
         <!-- extensions -->
         <xacro:endoscope_gazebo endoscope_name="${endoscope_name}"/>
-        <xacro:endoscope_transmission hardware_interface="${hardware_interface}" gripper_name="${endoscope_name}"/>
+        <xacro:endoscope_transmission hardware_interface="${hardware_interface}" endoscope_name="${endoscope_name}"/>
     </xacro:macro>
 </robot>
