Commit message: fixed typo

File: endoscope_description/urdf/endoscope.xacro (robot description, xacro)
@@ -32,5 +32,5 @@
         </link>
         <joint name="${endoscope_name}_joint_cm" type="fixed">
-            <parent link="${endsocope_name}_link_0"/>
+            <parent link="${endoscope_name}_link_0"/>
             <child link="${endoscope_name}_link_cm"/>
             <origin xyz="0 0 0.53186" rpy="0 0 0"/>

Commit message: removed transmission, as there are no joints

File: endoscope_description/urdf/endoscope.xacro (robot description, xacro)
@@ -1,9 +1,7 @@
 <?xml version="1.0"?>
 <robot xmlns:xacro="http://www.ros.org/wiki/xacro">
-    <xacro:macro name="endoscope" params="endoscope_name hardware_interface parent">
+    <xacro:macro name="endoscope" params="endoscope_name parent">
         <!-- include gazebo specifications -->
         <xacro:include filename="$(find endoscope_description)/urdf/endoscope.gazebo.xacro"/>
-        <!-- include transmission for ros_control -->
-        <xacro:include filename="$(find endoscope_description)/urdf/endoscope.transmission.xacro"/>
         <!--joint between {parent} and link_0-->
         <joint name="${parent}_${endoscope_name}_joint" type="fixed">
@@ -73,5 +71,4 @@
         <!-- extensions -->
         <xacro:endoscope_gazebo endoscope_name="${endoscope_name}"/>
-        <xacro:endoscope_transmission hardware_interface="${hardware_interface}" endoscope_name="${endoscope_name}"/>
     </xacro:macro>
 </robot>

Commit message: moved endoscope link position

File: endoscope_description/urdf/endoscope.xacro (robot description, xacro)
@@ -64,5 +64,5 @@
             <parent link="${endoscope_name}_link_1"/>
             <child link="${endoscope_name}_link_cm"/>
-            <origin xyz="0 0 0.53186" rpy="0 -1.57079632679 -1.57079632679"/>
+            <origin xyz="0 0 0.349946" rpy="0 -1.57079632679 -1.57079632679"/>
         </joint>
         <!-- camera link -->
