Commit message: added endoscope name and fixed typos

File: endoscope_description/urdf/endoscope.gazebo.xacro (robot description, xacro)
@@ -1,13 +1,13 @@
 <?xml version="1.0" ?>
 <robot xmlns:xacro="http://www.ros.org/wiki/xacro">
-  <xacro:macro name="endoscope_gazebo" params="robot_name"/>
+  <xacro:macro name="endoscope_gazebo" params="endoscope_name">
   <!-- ros_control-plugin -->
   <gazebo>
     <plugin filename="libgazebo_ros_control.so" name="control">
-      <robotNamespace>/${robot_name}</robotNamespace>
+      <robotNamespace>/${endoscope_name}</robotNamespace>
     </plugin>
   </gazebo>
   <!-- link 0 -->
-  <gazebo reference="link_0">
+  <gazebo reference="${endoscope_name}_link_0">
     <mu1>0.2</mu1>
     <mu2>0.2</mu2>

File: endoscope_description/urdf/endoscope.xacro (robot description, xacro)
@@ -1,35 +1,35 @@
 <?xml version="1.0"?>
 <robot xmlns:xacro="http://www.ros.org/wiki/xacro">
-    <xacro:macro name="endoscope" params="parent robot_name">
-    <!-- include gazebo specifications -->
-    <xacro:include filename="$(find endoscope_description)/urdf/endoscope.gazebo.xacro"/>
-    <!--joint between {parent} and link_0-->
-    <joint name="${parent}_${robot_name}_joint" type="fixed">
-        <parent link="${parent}"/>
-        <child link="link_0"/>
-    </joint>
-    <link name="link_0">
-        <inertial>
-            <origin rpy="0 0 0" xyz="-6.848375926496336e-18 3.4324719801768515e-07 0.11464386534267244"/>
-            <mass value="2.6062870546046777"/>
-            <inertia ixx="0.019428" ixy="-0.0" ixz="-0.0" iyy="0.019428" iyz="-0.0" izz="0.000824"/>
+    <xacro:macro name="endoscope" params="endoscope_name parent">
+        <!-- include gazebo specifications -->
+        <xacro:include filename="$(find endoscope_description)/urdf/endoscope.gazebo.xacro"/>
+        <!--joint between {parent} and link_0-->
+        <joint name="${parent}_${endoscope_name}_joint" type="fixed">
+            <parent link="${parent}"/>
+            <child link="${endoscope_name}_link_0"/>
+        </joint>
+        <link name="${endoscope_name}_link_0">
+            <inertial>
+                <origin rpy="0 0 0" xyz="-6.848375926496336e-18 3.4324719801768515e-07 0.11464386534267244"/>
+                <mass value="2.6062870546046777"/>
+                <inertia ixx="0.019428" ixy="-0.0" ixz="-0.0" iyy="0.019428" iyz="-0.0" izz="0.000824"/>
             </inertial>
-        <visual>
-            <origin rpy="0 0 0" xyz="0 0 0"/>
-            <geometry>
-                <mesh filename="package://endoscope_description/meshes/visual/link_0.stl"/>
-            </geometry>
-            <material name="silver">
-                <color rgba="1 0 0 1"/>
-            </material>
-        </visual>
-        <collision>
-            <origin rpy="0 0 0" xyz="0 0 0"/>
-            <geometry>
-                <mesh filename="package://endoscope_description/meshes/collisino/link_0.stl"/>
-            </geometry>
-        </collision>
-    </link>
-    <xacro:endoscope_gazebo robot_name="${robot_name}"/>
+            <visual>
+                <origin rpy="0 0 0" xyz="0 0 0"/>
+                <geometry>
+                    <mesh filename="package://endoscope_description/meshes/visual/link_0.stl"/>
+                </geometry>
+                <material name="silver">
+                    <color rgba="1 0 0 1"/>
+                </material>
+            </visual>
+            <collision>
+                <origin rpy="0 0 0" xyz="0 0 0"/>
+                <geometry>
+                    <mesh filename="package://endoscope_description/meshes/collision/link_0.stl"/>
+                </geometry>
+            </collision>
+        </link>
+        <xacro:endoscope_gazebo endoscope_name="${endoscope_name}"/>
     </xacro:macro>
 </robot>

Commit message: added camera plugin

File: endoscope_description/urdf/endoscope.gazebo.xacro (robot description, xacro)
@@ -1,18 +1,49 @@
 <?xml version="1.0" ?>
 <robot xmlns:xacro="http://www.ros.org/wiki/xacro">
-  <xacro:macro name="endoscope_gazebo" params="endoscope_name">
-  <!-- ros_control-plugin -->
-  <gazebo>
-    <plugin filename="libgazebo_ros_control.so" name="control">
-      <robotNamespace>/${endoscope_name}</robotNamespace>
-    </plugin>
-  </gazebo>
-  <!-- link 0 -->
-  <gazebo reference="${endoscope_name}_link_0">
-    <mu1>0.2</mu1>
-    <mu2>0.2</mu2>
-    <material>Gazebo/Grey</material>
-  </gazebo>
-  <!-- add camera -->
-  </xacro:macro>
+    <xacro:macro name="endoscope_gazebo" params="endoscope_name">
+    <!-- ros_control-plugin -->
+    <gazebo>
+        <plugin filename="libgazebo_ros_control.so" name="control">
+            <robotNamespace>/${endoscope_name}</robotNamespace>
+        </plugin>
+    </gazebo>
+    <!-- link 0 -->
+    <gazebo reference="${endoscope_name}_link_0">
+        <mu1>0.2</mu1>
+        <mu2>0.2</mu2>
+        <material>Gazebo/Grey</material>
+    </gazebo>
+    <!-- camera -->
+    <gazebo reference="${endoscope_name}_link_cm">
+        <sensor type="camera" name="${endoscope_name}_camera">
+            <update_rate>30.0</update_rate>
+            <camera name="head">
+                <horizontal_fov>1.3962634</horizontal_fov>
+                <image>
+                    <width>800</width>
+                    <height>800</height>
+                    <format>R8G8B8</format>
+                </image>
+                <clip>
+                    <near>0.02</near>
+                    <far>300</far>
+                </clip>
+            </camera>
+            <plugin name="camera_controller" filename="libgazebo_ros_camera.so">
+                <alwaysOn>true</alwaysOn>
+                <updateRate>0.0</updateRate>
+                <cameraName>${endoscope_name}/${endoscope_name}_camera</cameraName>
+                <imageTopicName>image_raw</imageTopicName>
+                <cameraInfoTopicName>camera_info</cameraInfoTopicName>
+                <frameName>camera_link</frameName>
+                <hackBaseline>0.07</hackBaseline>
+                <distortionK1>0.0</distortionK1>
+                <distortionK2>0.0</distortionK2>
+                <distortionK3>0.0</distortionK3>
+                <distortionT1>0.0</distortionT1>
+                <distortionT2>0.0</distortionT2>
+            </plugin>
+        </sensor>
+    </gazebo>
+    </xacro:macro>
 </robot>

File: endoscope_description/urdf/endoscope.xacro (robot description, xacro)
@@ -31,4 +31,12 @@
             </collision>
         </link>
+        <joint name="${endoscope_name}_joint_cm" type="fixed">
+            <parent link="${endsocope_name}_link_0"/>
+            <child link="${endoscope_name}_link_cm"/>
+            <origin xyz="0 0 0.53186" rpy="0 0 0"/>
+        </joint>
+        <link name="${endoscope_name}_link_cm">
+        </link>
+        <!-- extensions -->
         <xacro:endoscope_gazebo endoscope_name="${endoscope_name}"/>
     </xacro:macro>

Commit message: removed ros control plugin, rotated endoscope, changed endoscope resolution

File: endoscope_description/urdf/endoscope.gazebo.xacro (robot description, xacro)
@@ -2,10 +2,4 @@
 <robot xmlns:xacro="http://www.ros.org/wiki/xacro">
     <xacro:macro name="endoscope_gazebo" params="endoscope_name">
-    <!-- ros_control-plugin -->
-    <gazebo>
-        <plugin filename="libgazebo_ros_control.so" name="control">
-            <robotNamespace>/${endoscope_name}</robotNamespace>
-        </plugin>
-    </gazebo>
     <!-- link 0 -->
     <gazebo reference="${endoscope_name}_link_0">
@@ -21,6 +15,6 @@
                 <horizontal_fov>1.3962634</horizontal_fov>
                 <image>
-                    <width>800</width>
-                    <height>800</height>
+                    <width>320</width>
+                    <height>240</height>
                     <format>R8G8B8</format>
                 </image>
@@ -33,5 +27,5 @@
                 <alwaysOn>true</alwaysOn>
                 <updateRate>0.0</updateRate>
-                <cameraName>${endoscope_name}/${endoscope_name}_camera</cameraName>
+                <cameraName>${endoscope_name}_camera</cameraName>
                 <imageTopicName>image_raw</imageTopicName>
                 <cameraInfoTopicName>camera_info</cameraInfoTopicName>

File: endoscope_description/urdf/endoscope.xacro (robot description, xacro)
@@ -8,4 +8,5 @@
             <parent link="${parent}"/>
             <child link="${endoscope_name}_link_0"/>
+            <origin xyz="0 0 0" rpy="0 0 1.57079632679"/>
         </joint>
         <link name="${endoscope_name}_link_0">
@@ -34,5 +35,5 @@
             <parent link="${endoscope_name}_link_0"/>
             <child link="${endoscope_name}_link_cm"/>
-            <origin xyz="0 0 0.53186" rpy="0 0 0"/>
+            <origin xyz="0 0 0.53186" rpy="0 -1.57079632679 -1.57079632679"/>
         </joint>
         <link name="${endoscope_name}_link_cm">

Commit message: separated endoscope into two links

File: endoscope_description/urdf/endoscope.gazebo.xacro (robot description, xacro)
@@ -4,4 +4,10 @@
     <!-- link 0 -->
     <gazebo reference="${endoscope_name}_link_0">
+        <mu1>0.2</mu1>
+        <mu2>0.2</mu2>
+        <material>Gazebo/White</material>
+    </gazebo>
+    <!-- link 1 -->
+    <gazebo reference="${endoscope_name}_link_1">
         <mu1>0.2</mu1>
         <mu2>0.2</mu2>

File: endoscope_description/urdf/endoscope.xacro (robot description, xacro)
@@ -4,4 +4,6 @@
         <!-- include gazebo specifications -->
         <xacro:include filename="$(find endoscope_description)/urdf/endoscope.gazebo.xacro"/>
+        <!-- include transmission for ros_control -->
+        <xacro:include filename="$(find endoscope_description)/urdf/endoscope.transmission.xacro"/>
         <!--joint between {parent} and link_0-->
         <joint name="${parent}_${endoscope_name}_joint" type="fixed">
@@ -10,9 +12,10 @@
             <origin xyz="0 0 0" rpy="0 0 1.57079632679"/>
         </joint>
+        <!-- link 0 -->
         <link name="${endoscope_name}_link_0">
             <inertial>
-                <origin rpy="0 0 0" xyz="-6.848375926496336e-18 3.4324719801768515e-07 0.11464386534267244"/>
-                <mass value="2.6062870546046777"/>
-                <inertia ixx="0.019428" ixy="-0.0" ixz="-0.0" iyy="0.019428" iyz="-0.0" izz="0.000824"/>
+                <origin rpy="0 0 0" xyz="-7.270573632311392e-18 -7.270573632311392e-18 0.09976749827968114"/>
+                <mass value="2.4549415802586934"/>
+                <inertia ixx="0.008545" ixy="-0.0" ixz="-0.0" iyy="0.008545" iyz="-0.0" izz="0.000822"/>
             </inertial>
             <visual>
@@ -32,13 +35,43 @@
             </collision>
         </link>
+        <joint name="${endoscope_name}_joint_1" type="fixed">
+            <origin rpy="0 0 0" xyz="0.0 0.0 0.182"/>
+            <parent link="${endoscope_name}_link_0"/>
+            <child link="${endoscope_name}_link_1"/>
+        </joint>
+        <!-- link 1 -->
+        <link name="${endoscope_name}_link_1">
+            <inertial>
+                <origin rpy="0 0 0" xyz="-1.8420957352208925e-18 5.908967207684404e-06 0.17400951653092117"/>
+                <mass value="0.1513971388421877"/>
+                <inertia ixx="0.001529" ixy="-0.0" ixz="0.0" iyy="0.001529" iyz="-0.0" izz="1e-06"/>
+            </inertial>
+            <visual>
+                <origin rpy="0 0 0" xyz="0.0 -0.0 -0.182"/>
+                <geometry>
+                    <mesh filename="package://endoscope_description/meshes/visual/link_1.stl"/>
+                </geometry>
+                <material name="silver">
+                    <color rgba="1 0 0 1"/>
+                </material>
+            </visual>
+            <collision>
+                <origin rpy="0 0 0" xyz="0.0 -0.0 -0.182"/>
+                <geometry>
+                    <mesh filename="package://endoscope_description/meshes/collision/link_1.stl"/>
+                </geometry>
+            </collision>
+        </link>
         <joint name="${endoscope_name}_joint_cm" type="fixed">
-            <parent link="${endoscope_name}_link_0"/>
+            <parent link="${endoscope_name}_link_1"/>
             <child link="${endoscope_name}_link_cm"/>
             <origin xyz="0 0 0.53186" rpy="0 -1.57079632679 -1.57079632679"/>
         </joint>
+        <!-- camera link -->
         <link name="${endoscope_name}_link_cm">
         </link>
         <!-- extensions -->
         <xacro:endoscope_gazebo endoscope_name="${endoscope_name}"/>
+        <xacro:endoscope_transmission hardware_interface="${hardware_interface}" gripper_name="${endoscope_name}"/>
     </xacro:macro>
 </robot>

Commit message: added optical link

File: endoscope_description/urdf/endoscope.gazebo.xacro (robot description, xacro)
@@ -36,5 +36,5 @@
                 <imageTopicName>image_raw</imageTopicName>
                 <cameraInfoTopicName>camera_info</cameraInfoTopicName>
-                <frameName>camera_link</frameName>
+                <frameName>${endoscope_name}_link_cm_optical</frameName>
                 <hackBaseline>0.07</hackBaseline>
                 <distortionK1>0.0</distortionK1>

File: endoscope_description/urdf/endoscope.xacro (robot description, xacro)
@@ -69,4 +69,12 @@
         <link name="${endoscope_name}_link_cm">
         </link>
+        <!-- optical frame https://answers.ros.org/question/232534/gazebo-camera-frame-is-inconsistent-with-rviz-opencv-convention/ -->
+        <joint name="${endoscope_name}_joint_cm_optical" type="fixed">
+            <parent link="${endoscope_name}_link_cm"/>
+            <child link="${endoscope_name}_link_cm_optical"/>
+            <origin xyz="0 0 0" rpy="-1.57079632679 0 -1.57079632679"/>
+        </joint>
+        <link name="${endoscope_name}_link_cm_optical">
+        </link>
         <!-- extensions -->
         <xacro:endoscope_gazebo endoscope_name="${endoscope_name}"/>

Commit message: added robot_name to camera plugin

File: endoscope_description/urdf/endoscope.gazebo.xacro (robot description, xacro)
@@ -1,5 +1,5 @@
 <?xml version="1.0" ?>
 <robot xmlns:xacro="http://www.ros.org/wiki/xacro">
-    <xacro:macro name="endoscope_gazebo" params="endoscope_name">
+    <xacro:macro name="endoscope_gazebo" params="endoscope_name robot_name">
     <!-- link 0 -->
     <gazebo reference="${endoscope_name}_link_0">
@@ -33,4 +33,5 @@
                 <alwaysOn>true</alwaysOn>
                 <updateRate>0.0</updateRate>
+                <robotNamespace>/${robot_name}</robotNamespace>
                 <cameraName>${endoscope_name}_camera</cameraName>
                 <imageTopicName>image_raw</imageTopicName>

File: endoscope_description/urdf/endoscope.urdf.xacro (robot description, xacro)
@@ -6,7 +6,8 @@
     <!--  Arguments for the med7 macro  -->
     <xacro:arg name="endoscope_name" default="endoscope"/>
+    <xacro:arg name="robot_name" default="lbr"/>
     <!-- fix to world -->
     <link name="world"/>
     <!-- insert endoscope -->
-    <xacro:endoscope  endoscope_name="$(arg endoscope_name)" parent="world"/>
+    <xacro:endoscope  endoscope_name="$(arg endoscope_name)" robot_name="$(arg robot_name)" parent="world"/>
 </robot>

File: endoscope_description/urdf/endoscope.xacro (robot description, xacro)
@@ -1,5 +1,5 @@
 <?xml version="1.0"?>
 <robot xmlns:xacro="http://www.ros.org/wiki/xacro">
-    <xacro:macro name="endoscope" params="endoscope_name parent">
+    <xacro:macro name="endoscope" params="endoscope_name robot_name parent">
         <!-- include gazebo specifications -->
         <xacro:include filename="$(find endoscope_description)/urdf/endoscope.gazebo.xacro"/>
@@ -78,5 +78,5 @@
         </link>
         <!-- extensions -->
-        <xacro:endoscope_gazebo endoscope_name="${endoscope_name}"/>
+        <xacro:endoscope_gazebo endoscope_name="${endoscope_name}" robot_name="${robot_name}"/>
     </xacro:macro>
 </robot>
