Commit message: updated names

File: endoscope_description/urdf/endoscope.urdf.xacro (robot description, xacro)
@@ -3,5 +3,5 @@
 <robot xmlns:xacro="http://www.ros.org/wiki/xacro" name="endoscope">
     <!--Import the endoscope macro -->
-    <xacro:include filename="$(find endoscope_description)/urdf/endoscope.xacro"/>
+    <xacro:include filename="$(find da_vinci_endoscope_description)/urdf/endoscope.xacro"/>
     <!--  Arguments for the med7 macro  -->
     <xacro:arg name="endoscope_name" default="endoscope"/>

File: endoscope_description/urdf/endoscope.xacro (robot description, xacro)
@@ -3,5 +3,5 @@
     <xacro:macro name="endoscope" params="endoscope_name robot_name parent">
         <!-- include gazebo specifications -->
-        <xacro:include filename="$(find endoscope_description)/urdf/endoscope.gazebo.xacro"/>
+        <xacro:include filename="$(find da_vinci_endoscope_description)/urdf/endoscope.gazebo.xacro"/>
         <!--joint between {parent} and link_0-->
         <joint name="${parent}_${endoscope_name}_joint" type="fixed">
@@ -20,5 +20,5 @@
                 <origin rpy="0 0 0" xyz="0 0 0"/>
                 <geometry>
-                    <mesh filename="package://endoscope_description/meshes/visual/link_0.stl"/>
+                    <mesh filename="package://da_vinci_endoscope_description/meshes/visual/link_0.stl"/>
                 </geometry>
                 <material name="white">
@@ -29,5 +29,5 @@
                 <origin rpy="0 0 0" xyz="0 0 0"/>
                 <geometry>
-                    <mesh filename="package://endoscope_description/meshes/collision/link_0.stl"/>
+                    <mesh filename="package://da_vinci_endoscope_description/meshes/collision/link_0.stl"/>
                 </geometry>
             </collision>
@@ -48,5 +48,5 @@
                 <origin rpy="0 0 0" xyz="0.0 -0.0 -0.182"/>
                 <geometry>
-                    <mesh filename="package://endoscope_description/meshes/visual/link_1.stl"/>
+                    <mesh filename="package://da_vinci_endoscope_description/meshes/visual/link_1.stl"/>
                 </geometry>
                 <material name="silver">
@@ -57,5 +57,5 @@
                 <origin rpy="0 0 0" xyz="0.0 -0.0 -0.182"/>
                 <geometry>
-                    <mesh filename="package://endoscope_description/meshes/collision/link_1.stl"/>
+                    <mesh filename="package://da_vinci_endoscope_description/meshes/collision/link_1.stl"/>
                 </geometry>
             </collision>

File: gripper_description/urdf/gripper.urdf.xacro (robot description, xacro)
@@ -3,5 +3,5 @@
 <robot xmlns:xacro="http://www.ros.org/wiki/xacro" name="gripper">
     <!--Import the gripper macro -->
-    <xacro:include filename="$(find gripper_description)/urdf/gripper.xacro"/>
+    <xacro:include filename="$(find da_vinci_gripper_description)/urdf/gripper.xacro"/>
     <!--  Arguments for the med7 macro  -->
     <xacro:arg name="hardware_interface" default="PositionJointInterface"/>

File: gripper_description/urdf/gripper.xacro (robot description, xacro)
@@ -3,7 +3,7 @@
     <xacro:macro name="gripper" params="gripper_name hardware_interface parent">
         <!-- include gazebo specifications -->
-        <xacro:include filename="$(find gripper_description)/urdf/gripper.gazebo.xacro"/>
+        <xacro:include filename="$(find da_vinci_gripper_description)/urdf/gripper.gazebo.xacro"/>
         <!-- include transmission for ros_control -->
-        <xacro:include filename="$(find gripper_description)/urdf/gripper.transmission.xacro"/>
+        <xacro:include filename="$(find da_vinci_gripper_description)/urdf/gripper.transmission.xacro"/>
         <!--joint between {parent} and link_0-->
         <joint name="${parent}_${gripper_name}_joint" type="fixed">
@@ -21,5 +21,5 @@
                 <origin rpy="0 0 0" xyz="0 0 0"/>
                 <geometry>
-                    <mesh filename="package://gripper_description/meshes/visual/link_0.stl"/>
+                    <mesh filename="package://da_vinci_gripper_description/meshes/visual/link_0.stl"/>
                 </geometry>
                 <material name="silver">
@@ -30,5 +30,5 @@
                 <origin rpy="0 0 0" xyz="0 0 0"/>
                 <geometry>
-                    <mesh filename="package://gripper_description/meshes/collision/link_0.stl"/>
+                    <mesh filename="package://da_vinci_gripper_description/meshes/collision/link_0.stl"/>
                 </geometry>
             </collision>
@@ -49,5 +49,5 @@
                 <origin rpy="0 0 0" xyz="0.0 0.417886 -0.064767"/>
                 <geometry>
-                    <mesh filename="package://gripper_description/meshes/visual/link_1.stl"/>
+                    <mesh filename="package://da_vinci_gripper_description/meshes/visual/link_1.stl"/>
                 </geometry>
                 <material name="silver">
@@ -58,5 +58,5 @@
                 <origin rpy="0 0 0" xyz="0.0 0.417886 -0.064767"/>
                 <geometry>
-                    <mesh filename="package://gripper_description/meshes/collision/link_1.stl"/>
+                    <mesh filename="package://da_vinci_gripper_description/meshes/collision/link_1.stl"/>
                 </geometry>
             </collision>
@@ -78,5 +78,5 @@
                 <origin rpy="0 0 0" xyz="-0.004011 0.426986 -0.064842"/>
                 <geometry>
-                    <mesh filename="package://gripper_description/meshes/visual/link_2.stl"/>
+                    <mesh filename="package://da_vinci_gripper_description/meshes/visual/link_2.stl"/>
                 </geometry>
                 <material name="silver">
@@ -87,5 +87,5 @@
                 <origin rpy="0 0 0" xyz="-0.004011 0.426986 -0.064842"/>
                 <geometry>
-                    <mesh filename="package://gripper_description/meshes/collision/link_2.stl"/>
+                    <mesh filename="package://da_vinci_gripper_description/meshes/collision/link_2.stl"/>
                 </geometry>
             </collision>
@@ -107,5 +107,5 @@
                 <origin rpy="0 0 0" xyz="-1.6e-05 0.43587 -0.066816"/>
                 <geometry>
-                    <mesh filename="package://gripper_description/meshes/visual/link_3.stl"/>
+                    <mesh filename="package://da_vinci_gripper_description/meshes/visual/link_3.stl"/>
                 </geometry>
                 <material name="silver">
@@ -116,5 +116,5 @@
                 <origin rpy="0 0 0" xyz="-1.6e-05 0.43587 -0.066816"/>
                 <geometry>
-                    <mesh filename="package://gripper_description/meshes/collision/link_3.stl"/>
+                    <mesh filename="package://da_vinci_gripper_description/meshes/collision/link_3.stl"/>
                 </geometry>
             </collision>
@@ -136,5 +136,5 @@
                 <origin rpy="0 0 0" xyz="1.7e-05 0.435902 -0.062916"/>
                 <geometry>
-                    <mesh filename="package://gripper_description/meshes/visual/link_4.stl"/>
+                    <mesh filename="package://da_vinci_gripper_description/meshes/visual/link_4.stl"/>
                 </geometry>
                 <material name="silver">
@@ -145,5 +145,5 @@
                 <origin rpy="0 0 0" xyz="1.7e-05 0.435902 -0.062916"/>
                 <geometry>
-                    <mesh filename="package://gripper_description/meshes/collision/link_4.stl"/>
+                    <mesh filename="package://da_vinci_gripper_description/meshes/collision/link_4.stl"/>
                 </geometry>
             </collision>
