Commit message: renamed and removed links

File: storz_endoscope_description/urdf/endoscope.xacro (robot description, xacro)
@@ -44,24 +44,5 @@
   </collision>
 </link>
-<link name="virtual_camera_link_1">
-  <inertial>
-    <origin rpy="0 0 0" xyz="0.0002500000000000002 -2.0895063973251776e-13 -1.9359513991901167e-15"/>
-    <mass value="4.9323004661359056e-05"/>
-    <inertia ixx="0.0" ixy="0.0" ixz="0.0" iyy="0.0" iyz="0.0" izz="0.0"/>
-  </inertial>
-  <visual>
-    <origin rpy="0 0 0" xyz="0.1903 -0.0 -0.0415"/>
-    <geometry>
-      <mesh filename="package://storz_endoscope_description/meshes/virtual_camera_link_1.stl" scale="0.001 0.001 0.001"/>
-    </geometry>
-    <material name="silver"/>
-  </visual>
-  <collision>
-    <origin rpy="0 0 0" xyz="0.1903 -0.0 -0.0415"/>
-    <geometry>
-      <mesh filename="package://storz_endoscope_description/meshes/virtual_camera_link_1.stl" scale="0.001 0.001 0.001"/>
-    </geometry>
-  </collision>
-</link>
+<link name="virtual_camera_link_1"/>
 <joint name="Rigid1" type="fixed">
   <origin rpy="0 0 0" xyz="0.0433 0.0 0.0415"/>
