Commit message: merged un moveable links

File: storz_endoscope_description/urdf/storz_endoscope.gazebo.xacro (robot description, xacro)
@@ -4,10 +4,4 @@
         <!-- link 0 -->
         <gazebo reference="link_0">
-            <mu1>0.2</mu1>
-            <mu2>0.2</mu2>
-            <material>Gazebo/Grey</material>
-        </gazebo>
-        <!-- link 1 -->
-        <gazebo reference="link_1">
             <mu1>0.2</mu1>
             <mu2>0.2</mu2>

File: storz_endoscope_description/urdf/storz_endoscope.xacro (robot description, xacro)
@@ -8,5 +8,5 @@
             <parent link="${parent}"/>
             <child link="${endoscope_name}_link_0"/>
-            <origin xyz="0 0 0" rpy="0 0 0"/>
+            <origin xyz="0 0 0" rpy="0 0 1.57079632679"/>
         </joint>
         <!-- link 0 -->
@@ -33,32 +33,4 @@
             </collision>
         </link>
-        <joint name="${endoscope_name}_joint_1" type="fixed">
-            <origin rpy="0 0 0" xyz="0.0433 0.0 0.0415"/>
-            <parent link="${endoscope_name}_link_0"/>
-            <child link="${endoscope_name}_link_1"/>
-        </joint>
-        <!-- link 1 -->
-        <link name="${endoscope_name}_link_1">
-            <inertial>
-                <origin rpy="0 0 0" xyz="0.046573718971088175 -0.0015143640659485344 -4.88787786356859e-07"/>
-                <mass value="0.9169103264945898"/>
-                <inertia ixx="0.000214" ixy="5.5e-05" ixz="-0.0" iyy="0.000789" iyz="0.0" izz="0.000835"/>
-            </inertial>
-            <visual>
-                <origin rpy="0 0 0" xyz="-0.0433 0.0 -0.0415"/>
-                <geometry>
-                    <mesh filename="package://storz_endoscope_description/meshes/visual/link_1.stl" scale="0.001 0.001 0.001"/>
-                </geometry>
-                <material name="silver">
-                    <color rgba="1 0 0 1"/>
-                </material>
-            </visual>
-            <collision>
-                <origin rpy="0 0 0" xyz="-0.0433 0.0 -0.0415"/>
-                <geometry>
-                    <mesh filename="package://storz_endoscope_description/meshes/collision/link_1.stl" scale="0.001 0.001 0.001"/>
-                </geometry>
-            </collision>
-        </link>
         <joint name="${endoscope_name}_joint_cm" type="fixed">
             <origin rpy="0 0 0" xyz="-0.1903 0.0 0.0415"/>

Commit message: added link 1 to storz endoscope

File: storz_endoscope_description/urdf/storz_endoscope.gazebo.xacro (robot description, xacro)
@@ -4,4 +4,10 @@
         <!-- link 0 -->
         <gazebo reference="link_0">
+            <mu1>0.2</mu1>
+            <mu2>0.2</mu2>
+            <material>Gazebo/Grey</material>
+        </gazebo>
+        <!-- link 1 -->
+        <gazebo reference="link_1">
             <mu1>0.2</mu1>
             <mu2>0.2</mu2>
