Commit message: finished storz endoscope

File: storz_endoscope_description/urdf/storz_endoscope.xacro (robot description, xacro)
@@ -1,56 +1,81 @@
 <?xml version="1.0" ?>
-<robot name="endoscope" xmlns:xacro="http://www.ros.org/wiki/xacro">
-<xacro:include filename="$(find storz_endoscope_description)/urdf/materials.xacro" />
-<xacro:include filename="$(find storz_endoscope_description)/urdf/storz_endoscope.gazebo" />
-<link name="link_0">
-  <inertial>
-    <origin rpy="0 0 0" xyz="0.0011044635060518421 -0.00025940397558044673 0.024608364371170997"/>
-    <mass value="0.6888304856441179"/>
-    <inertia ixx="0.000315" ixy="-0.0" ixz="-1.3e-05" iyy="0.000607" iyz="3e-06" izz="0.000517"/>
-  </inertial>
-  <visual>
-    <origin rpy="0 0 0" xyz="0 0 0"/>
-    <geometry>
-      <mesh filename="package://storz_endoscope_description/meshes/link_0.stl" scale="0.001 0.001 0.001"/>
-    </geometry>
-    <material name="silver"/>
-  </visual>
-  <collision>
-    <origin rpy="0 0 0" xyz="0 0 0"/>
-    <geometry>
-      <mesh filename="package://storz_endoscope_description/meshes/link_0.stl" scale="0.001 0.001 0.001"/>
-    </geometry>
-  </collision>
-</link>
-<link name="link_1">
-  <inertial>
-    <origin rpy="0 0 0" xyz="0.046573718971088175 -0.0015143640659485344 -4.88787786356859e-07"/>
-    <mass value="0.9169103264945898"/>
-    <inertia ixx="0.000214" ixy="5.5e-05" ixz="-0.0" iyy="0.000789" iyz="0.0" izz="0.000835"/>
-  </inertial>
-  <visual>
-    <origin rpy="0 0 0" xyz="-0.0433 0.0 -0.0415"/>
-    <geometry>
-      <mesh filename="package://storz_endoscope_description/meshes/link_1.stl" scale="0.001 0.001 0.001"/>
-    </geometry>
-    <material name="silver"/>
-  </visual>
-  <collision>
-    <origin rpy="0 0 0" xyz="-0.0433 0.0 -0.0415"/>
-    <geometry>
-      <mesh filename="package://storz_endoscope_description/meshes/link_1.stl" scale="0.001 0.001 0.001"/>
-    </geometry>
-  </collision>
-</link>
-<link name="virtual_camera_link_1"/>
-<joint name="Rigid1" type="fixed">
-  <origin rpy="0 0 0" xyz="0.0433 0.0 0.0415"/>
-  <parent link="link_0"/>
-  <child link="link_1"/>
-</joint>
-<joint name="Rigid2" type="fixed">
-  <origin rpy="0 0 0" xyz="-0.1903 0.0 0.0415"/>
-  <parent link="link_0"/>
-  <child link="virtual_camera_link_1"/>
-</joint>
+<robot xmlns:xacro="http://www.ros.org/wiki/xacro">
+    <xacro:macro name="storz_endoscope" params="endoscope_name robot_name parent">
+        <!-- include gazebo specifications -->
+        <xacro:include filename="$(find storz_endoscope_description)/urdf/storz_endoscope.gazebo.xacro" />
+        <!--joint between {parent} and link_0-->
+        <joint name="${parent}_${endoscope_name}_joint" type="fixed">
+            <parent link="${parent}"/>
+            <child link="${endoscope_name}_link_0"/>
+            <origin xyz="0 0 0" rpy="0 0 0"/>
+        </joint>
+        <!-- link 0 -->
+        <link name="${endoscope_name}_link_0">
+            <inertial>
+                <origin rpy="0 0 0" xyz="0.0011044635060518421 -0.00025940397558044673 0.024608364371170997"/>
+                <mass value="0.6888304856441179"/>
+                <inertia ixx="0.000315" ixy="-0.0" ixz="-1.3e-05" iyy="0.000607" iyz="3e-06" izz="0.000517"/>
+            </inertial>
+            <visual>
+                <origin rpy="0 0 0" xyz="0 0 0"/>
+                <geometry>
+                    <mesh filename="package://storz_endoscope_description/meshes/visual/link_0.stl" scale="0.001 0.001 0.001"/>
+                </geometry>
+                <material name="silver">
+                    <color rgba="1 0 0 1"/>
+                </material>
+            </visual>
+            <collision>
+                <origin rpy="0 0 0" xyz="0 0 0"/>
+                <geometry>
+                    <mesh filename="package://storz_endoscope_description/meshes/collision/link_0.stl" scale="0.001 0.001 0.001"/>
+                </geometry>
+            </collision>
+        </link>
+        <joint name="${endoscope_name}_joint_1" type="fixed">
+            <origin rpy="0 0 0" xyz="0.0433 0.0 0.0415"/>
+            <parent link="${endoscope_name}_link_0"/>
+            <child link="${endoscope_name}_link_1"/>
+        </joint>
+        <!-- link 1 -->
+        <link name="${endoscope_name}_link_1">
+            <inertial>
+                <origin rpy="0 0 0" xyz="0.046573718971088175 -0.0015143640659485344 -4.88787786356859e-07"/>
+                <mass value="0.9169103264945898"/>
+                <inertia ixx="0.000214" ixy="5.5e-05" ixz="-0.0" iyy="0.000789" iyz="0.0" izz="0.000835"/>
+            </inertial>
+            <visual>
+                <origin rpy="0 0 0" xyz="-0.0433 0.0 -0.0415"/>
+                <geometry>
+                    <mesh filename="package://storz_endoscope_description/meshes/visual/link_1.stl" scale="0.001 0.001 0.001"/>
+                </geometry>
+                <material name="silver">
+                    <color rgba="1 0 0 1"/>
+                </material>
+            </visual>
+            <collision>
+                <origin rpy="0 0 0" xyz="-0.0433 0.0 -0.0415"/>
+                <geometry>
+                    <mesh filename="package://storz_endoscope_description/meshes/collision/link_1.stl" scale="0.001 0.001 0.001"/>
+                </geometry>
+            </collision>
+        </link>
+        <joint name="${endoscope_name}_joint_cm" type="fixed">
+            <origin rpy="0 0 0" xyz="-0.1903 0.0 0.0415"/>
+            <parent link="${endoscope_name}_link_0"/>
+            <child link="${endoscope_name}_link_cm"/>
+        </joint>
+        <!-- camera link -->
+        <link name="${endoscope_name}_link_cm"/>
+        <!-- optical frame https://answers.ros.org/question/232534/gazebo-camera-frame-is-inconsistent-with-rviz-opencv-convention/ -->
+        <joint name="${endoscope_name}_joint_cm_optical" type="fixed">
+            <parent link="${endoscope_name}_link_cm"/>
+            <child link="${endoscope_name}_link_cm_optical"/>
+            <origin xyz="0 0 0" rpy="-1.57079632679 0 -1.57079632679"/>
+        </joint>
+        <link name="${endoscope_name}_link_cm_optical">
+        </link>
+        <!-- extensions -->
+        <xacro:storz_endoscope_gazebo endoscope_name="${endoscope_name}" robot_name="${robot_name}"/>
+    </xacro:macro>
 </robot>

Commit message: updated camera orientation

File: storz_endoscope_description/urdf/storz_endoscope.xacro (robot description, xacro)
@@ -34,5 +34,5 @@
         </link>
         <joint name="${endoscope_name}_joint_cm" type="fixed">
-            <origin rpy="0 0 0" xyz="-0.1903 0.0 0.0415"/>
+            <origin rpy="1.57079632679 0 3.141592654" xyz="-0.1903 0.0 0.0415"/>
             <parent link="${endoscope_name}_link_0"/>
             <child link="${endoscope_name}_link_cm"/>

Commit message: added link_1 to storz endoscope

File: storz_endoscope_description/urdf/storz_endoscope.xacro (robot description, xacro)
@@ -13,7 +13,7 @@
         <link name="${endoscope_name}_link_0">
             <inertial>
-                <origin rpy="0 0 0" xyz="0.0011044635060518421 -0.00025940397558044673 0.024608364371170997"/>
-                <mass value="0.6888304856441179"/>
-                <inertia ixx="0.000315" ixy="-0.0" ixz="-1.3e-05" iyy="0.000607" iyz="3e-06" izz="0.000517"/>
+                <origin rpy="0 0 0" xyz="0.05347530282631193 -0.0009866876037994033 0.03417463143575086"/>
+                <mass value="1.5884453511086485"/>
+                <inertia ixx="0.000641" ixy="9.6e-05" ixz="-0.000622" iyy="0.004145" iyz="1.2e-05" izz="0.003991"/>
             </inertial>
             <visual>
@@ -29,11 +29,39 @@
                 <origin rpy="0 0 0" xyz="0 0 0"/>
                 <geometry>
-                    <mesh filename="package://storz_endoscope_description/meshes/collision/link_0.stl" scale="0.001 0.001 0.001"/>
+                <mesh filename="package://storz_endoscope_description/meshes/collision/link_0.stl" scale="0.001 0.001 0.001"/>
+                </geometry>
+            </collision>
+        </link>
+        <joint name="${endoscope_name}_joint_1" type="fixed">
+            <origin rpy="0 0 0" xyz="-0.015 0.0 0.0415"/>
+            <parent link="${endoscope_name}_link_0"/>
+            <child link="${endoscope_name}_link_1"/>
+        </joint>
+        <!-- link 1 -->
+        <link name="${endoscope_name}_link_1">
+            <inertial>
+                <origin rpy="0 0 0" xyz="-0.08761286703720295 1.6070339520327724e-16 2.081251837537934e-13"/>
+                <mass value="0.017299976665697662"/>
+                <inertia ixx="0.0" ixy="-0.0" ixz="-0.0" iyy="4.4e-05" iyz="-0.0" izz="4.4e-05"/>
+            </inertial>
+            <visual>
+                <origin rpy="0 0 0" xyz="0.015 -0.0 -0.0415"/>
+                <geometry>
+                    <mesh filename="package://storz_endoscope_description/meshes/visual/link_1.stl" scale="0.001 0.001 0.001"/>
+                </geometry>
+                <material name="silver">
+                    <color rgba="1 0 0 1"/>
+                </material>
+            </visual>
+            <collision>
+                <origin rpy="0 0 0" xyz="0.015 -0.0 -0.0415"/>
+                <geometry>
+                    <mesh filename="package://storz_endoscope_description/meshes/collision/link_1.stl" scale="0.001 0.001 0.001"/>
                 </geometry>
             </collision>
         </link>
         <joint name="${endoscope_name}_joint_cm" type="fixed">
-            <origin rpy="1.57079632679 0 3.141592654" xyz="-0.1903 0.0 0.0415"/>
-            <parent link="${endoscope_name}_link_0"/>
+            <origin rpy="1.57079632679 0 3.141592654" xyz="-0.1753 0.0 0.0"/>
+            <parent link="${endoscope_name}_link_1"/>
             <child link="${endoscope_name}_link_cm"/>
         </joint>

Commit message: changed initial angle

File: storz_endoscope_description/urdf/storz_endoscope.xacro (robot description, xacro)
@@ -8,5 +8,5 @@
             <parent link="${parent}"/>
             <child link="${endoscope_name}_link_0"/>
-            <origin xyz="0 0 0" rpy="0 0 1.57079632679"/>
+            <origin xyz="0 0 0" rpy="0 0 3.141592654"/>
         </joint>
         <!-- link 0 -->
@@ -69,8 +69,9 @@
         <link name="${endoscope_name}_link_cm"/>
         <!-- optical frame https://answers.ros.org/question/232534/gazebo-camera-frame-is-inconsistent-with-rviz-opencv-convention/ -->
-        <joint name="${endoscope_name}_joint_cm_optical" type="fixed">
+        <joint name="${endoscope_name}_joint_cm_optical" type="fixed">  <!-- add continuous joint to rotate image digitally -->
             <parent link="${endoscope_name}_link_cm"/>
             <child link="${endoscope_name}_link_cm_optical"/>
             <origin xyz="0 0 0" rpy="-1.57079632679 0 -1.57079632679"/>
+            <!--axis xyz="0.0 0.0 0.01"/-->  <!-- rotate about the optical axis -->
         </joint>
         <link name="${endoscope_name}_link_cm_optical">

Commit message: reset endoscope orientation

File: storz_endoscope_description/urdf/storz_endoscope.xacro (robot description, xacro)
@@ -8,5 +8,5 @@
             <parent link="${parent}"/>
             <child link="${endoscope_name}_link_0"/>
-            <origin xyz="0 0 0" rpy="0 0 3.141592654"/>
+            <origin xyz="0 0 0" rpy="0 0 1.57079632679"/>
         </joint>
         <!-- link 0 -->
