Commit message: updated name

File: da_vinci_endoscope_description/urdf/da_vinci_endoscope.gazebo.xacro (robot description, xacro)
@@ -1,5 +1,5 @@
 <?xml version="1.0" ?>
 <robot xmlns:xacro="http://www.ros.org/wiki/xacro">
-    <xacro:macro name="endoscope_gazebo" params="endoscope_name robot_name">
+    <xacro:macro name="da_vinci_endoscope_gazebo" params="endoscope_name robot_name">
     <!-- link 0 -->
     <gazebo reference="${endoscope_name}_link_0">

File: da_vinci_endoscope_description/urdf/da_vinci_endoscope.urdf.xacro (robot description, xacro)
@@ -10,4 +10,4 @@
     <link name="world"/>
     <!-- insert endoscope -->
-    <xacro:endoscope  endoscope_name="$(arg endoscope_name)" robot_name="$(arg robot_name)" parent="world"/>
+    <xacro:da_vinci_endoscope  endoscope_name="$(arg endoscope_name)" robot_name="$(arg robot_name)" parent="world"/>
 </robot>

File: da_vinci_endoscope_description/urdf/da_vinci_endoscope.xacro (robot description, xacro)
@@ -1,5 +1,5 @@
 <?xml version="1.0"?>
 <robot xmlns:xacro="http://www.ros.org/wiki/xacro">
-    <xacro:macro name="endoscope" params="endoscope_name robot_name parent">
+    <xacro:macro name="da_vinci_endoscope" params="endoscope_name robot_name parent">
         <!-- include gazebo specifications -->
         <xacro:include filename="$(find da_vinci_endoscope_description)/urdf/da_vinci_endoscope.gazebo.xacro"/>
@@ -78,5 +78,5 @@
         </link>
         <!-- extensions -->
-        <xacro:endoscope_gazebo endoscope_name="${endoscope_name}" robot_name="${robot_name}"/>
+        <xacro:da_vinci_endoscope_gazebo endoscope_name="${endoscope_name}" robot_name="${robot_name}"/>
     </xacro:macro>
 </robot>

Commit message: updated gazebo

File: da_vinci_endoscope_description/urdf/da_vinci_endoscope.gazebo.xacro (robot description, xacro)
@@ -2,49 +2,49 @@
 <robot xmlns:xacro="http://www.ros.org/wiki/xacro">
     <xacro:macro name="da_vinci_endoscope_gazebo" params="endoscope_name robot_name">
-    <!-- link 0 -->
-    <gazebo reference="${endoscope_name}_link_0">
-        <mu1>0.2</mu1>
-        <mu2>0.2</mu2>
-        <material>Gazebo/White</material>
-    </gazebo>
-    <!-- link 1 -->
-    <gazebo reference="${endoscope_name}_link_1">
-        <mu1>0.2</mu1>
-        <mu2>0.2</mu2>
-        <material>Gazebo/Grey</material>
-    </gazebo>
-    <!-- camera -->
-    <gazebo reference="${endoscope_name}_link_cm">
-        <sensor type="camera" name="${endoscope_name}_camera">
-            <update_rate>30.0</update_rate>
-            <camera name="head">
-                <horizontal_fov>1.3962634</horizontal_fov>
-                <image>
-                    <width>320</width>
-                    <height>240</height>
-                    <format>R8G8B8</format>
-                </image>
-                <clip>
-                    <near>0.02</near>
-                    <far>300</far>
-                </clip>
-            </camera>
-            <plugin name="camera_controller" filename="libgazebo_ros_camera.so">
-                <alwaysOn>true</alwaysOn>
-                <updateRate>0.0</updateRate>
-                <robotNamespace>/${robot_name}</robotNamespace>
-                <cameraName>${endoscope_name}_camera</cameraName>
-                <imageTopicName>image_raw</imageTopicName>
-                <cameraInfoTopicName>camera_info</cameraInfoTopicName>
-                <frameName>${endoscope_name}_link_cm_optical</frameName>
-                <hackBaseline>0.07</hackBaseline>
-                <distortionK1>0.0</distortionK1>
-                <distortionK2>0.0</distortionK2>
-                <distortionK3>0.0</distortionK3>
-                <distortionT1>0.0</distortionT1>
-                <distortionT2>0.0</distortionT2>
-            </plugin>
-        </sensor>
-    </gazebo>
+        <!-- link 0 -->
+        <gazebo reference="${endoscope_name}_link_0">
+            <mu1>0.2</mu1>
+            <mu2>0.2</mu2>
+            <material>Gazebo/White</material>
+        </gazebo>
+        <!-- link 1 -->
+        <gazebo reference="${endoscope_name}_link_1">
+            <mu1>0.2</mu1>
+            <mu2>0.2</mu2>
+            <material>Gazebo/Grey</material>
+        </gazebo>
+        <!-- camera -->
+        <gazebo reference="${endoscope_name}_link_cm">
+            <sensor type="camera" name="${endoscope_name}_camera">
+                <update_rate>30.0</update_rate>
+                <camera name="head">
+                    <horizontal_fov>1.3962634</horizontal_fov>
+                    <image>
+                        <width>320</width>
+                        <height>240</height>
+                        <format>R8G8B8</format>
+                    </image>
+                    <clip>
+                        <near>0.02</near>
+                        <far>300</far>
+                    </clip>
+                </camera>
+                <plugin name="camera_controller" filename="libgazebo_ros_camera.so">
+                    <alwaysOn>true</alwaysOn>
+                    <updateRate>0.0</updateRate>
+                    <robotNamespace>/${robot_name}</robotNamespace>
+                    <cameraName>${endoscope_name}_camera</cameraName>
+                    <imageTopicName>image_raw</imageTopicName>
+                    <cameraInfoTopicName>camera_info</cameraInfoTopicName>
+                    <frameName>${endoscope_name}_link_cm_optical</frameName>
+                    <hackBaseline>0.07</hackBaseline>
+                    <distortionK1>0.0</distortionK1>
+                    <distortionK2>0.0</distortionK2>
+                    <distortionK3>0.0</distortionK3>
+                    <distortionT1>0.0</distortionT1>
+                    <distortionT2>0.0</distortionT2>
+                </plugin>
+            </sensor>
+        </gazebo>
     </xacro:macro>
 </robot>

File: storz_endoscope_description/urdf/storz_endoscope.gazebo.xacro (robot description, xacro)
@@ -3,5 +3,5 @@
     <xacro:macro name="storz_endoscope_gazebo" params="endoscope_name robot_name">
         <!-- link 0 -->
-        <gazebo reference="link_0">
+        <gazebo reference="${endoscope_name}_link_0">
             <mu1>0.2</mu1>
             <mu2>0.2</mu2>
@@ -9,5 +9,5 @@
         </gazebo>
         <!-- link 1 -->
-        <gazebo reference="link_1">
+        <gazebo reference="${endoscope_name}_link_1">
             <mu1>0.2</mu1>
             <mu2>0.2</mu2>
