Commit message: added env hook and moved gazebo

File: da_vinci_endoscope_description/urdf/da_vinci_endoscope_description.urdf.xacro (robot description, xacro)
@@ -3,5 +3,5 @@
     <xacro:macro name="da_vinci_endoscope" params="endoscope_name robot_name parent">
         <!-- include gazebo specifications -->
-        <xacro:include filename="$(find da_vinci_endoscope_description)/urdf/da_vinci_endoscope.gazebo.xacro"/>
+        <xacro:include filename="$(find da_vinci_endoscope_description)/gazebo/da_vinci_endoscope.gazebo.xacro"/>
         <!--joint between {parent} and link_0-->
         <joint name="${parent}_${endoscope_name}_joint" type="fixed">

File: storz_endoscope_description/urdf/storz_endoscope_description.urdf.xacro (robot description, xacro)
@@ -3,5 +3,5 @@
     <xacro:macro name="storz_endoscope" params="endoscope_name robot_name parent">
         <!-- include gazebo specifications -->
-        <xacro:include filename="$(find storz_endoscope_description)/urdf/storz_endoscope.gazebo.xacro" />
+        <xacro:include filename="$(find storz_endoscope_description)/gazebo/storz_endoscope.gazebo.xacro" />
         <!--joint between {parent} and link_0-->
         <joint name="${parent}_${endoscope_name}_joint" type="fixed">

File: storz_exoscope_description/urdf/storz_exoscope_description.urdf.xacro (robot description, xacro)
@@ -1,7 +1,7 @@
 <?xml version="1.0" ?>
 <robot xmlns:xacro="http://www.ros.org/wiki/xacro">
-    <xacro:macro name="storz_straight_exoscope_hsi" params="exoscope_name robot_name parent">
+    <xacro:macro name="storz_exoscope" params="exoscope_name robot_name parent">
         <!-- include gazebo specifications -->
-        <xacro:include filename="$(find storz_straight_exoscope_hsi_description)/urdf/storz_straight_exoscope_hsi.gazebo.xacro" />
+        <xacro:include filename="$(find storz_exoscope_description)/gazebo/storz_exoscope.gazebo.xacro" />
         <!--joint between {parent} and link_0-->
         <joint name="${parent}_${exoscope_name}_joint" type="fixed">
@@ -13,12 +13,12 @@
         <link name="${exoscope_name}_link_0">
             <inertial>
-                <origin rpy="0 0 0" xyz="0.04071287283172147 -8.153806755863768e-05 -0.04195721621845735"/>
-                <mass value="2.4245187944339057"/>
-                <inertia ixx="0.00996" ixy="1e-06" ixz="0.000598" iyy="0.01031" iyz="0.000146" izz="0.00104"/>
+                <origin rpy="0 0 0" xyz="0.03997881004884705 -0.0005082075189353901 -0.03926307553084657"/>
+                <mass value="2.1436339240369744"/>
+                <inertia ixx="0.008938" ixy="7e-06" ixz="0.000553" iyy="0.009241" iyz="-0.000113" izz="0.000887"/>
             </inertial>
             <visual>
                 <origin rpy="0 0 0" xyz="0 0 0"/>
                 <geometry>
-                    <mesh filename="package://storz_straight_exoscope_hsi_description/meshes/visual/link_0.stl" scale="0.001 0.001 0.001"/>
+                    <mesh filename="package://storz_exoscope_description/meshes/visual/link_0.stl" scale="0.001 0.001 0.001"/>
                 </geometry>
                 <material name="silver">
@@ -29,10 +29,10 @@
                 <origin rpy="0 0 0" xyz="0 0 0"/>
                 <geometry>
-                    <mesh filename="package://storz_straight_exoscope_hsi_description/meshes/collision/link_0.stl" scale="0.001 0.001 0.001"/>
+                    <mesh filename="package://storz_exoscope_description/meshes/collision/link_0.stl" scale="0.001 0.001 0.001"/>
                 </geometry>
             </collision>
         </link>
         <joint name="${exoscope_name}_joint_cm" type="fixed">
-            <origin rpy="-1.57079632679 -1.57079632679 0" xyz="0.046594 0.000596 0.1205"/>
+            <origin rpy="0 0 -1.57079632679" xyz="0.047 -0.005826 0.115248"/>
             <parent link="${exoscope_name}_link_0"/>
             <child link="${exoscope_name}_link_cm"/>
@@ -50,5 +50,5 @@
         </link>
         <!-- extensions -->
-        <xacro:storz_straight_exoscope_hsi_gazebo exoscope_name="${exoscope_name}" robot_name="${robot_name}"/>
+        <xacro:storz_exoscope_gazebo exoscope_name="${exoscope_name}" robot_name="${robot_name}"/>
     </xacro:macro>
 </robot>

File: storz_straight_exoscope_hsi_description/urdf/storz_straight_exoscope_hsi_description.urdf.xacro (robot description, xacro)
@@ -1,7 +1,7 @@
 <?xml version="1.0" ?>
 <robot xmlns:xacro="http://www.ros.org/wiki/xacro">
-    <xacro:macro name="storz_exoscope" params="exoscope_name robot_name parent">
+    <xacro:macro name="storz_straight_exoscope_hsi" params="exoscope_name robot_name parent">
         <!-- include gazebo specifications -->
-        <xacro:include filename="$(find storz_exoscope_description)/urdf/storz_exoscope.gazebo.xacro" />
+        <xacro:include filename="$(find storz_straight_exoscope_hsi_description)/gazebo/storz_straight_exoscope_hsi.gazebo.xacro" />
         <!--joint between {parent} and link_0-->
         <joint name="${parent}_${exoscope_name}_joint" type="fixed">
@@ -13,12 +13,12 @@
         <link name="${exoscope_name}_link_0">
             <inertial>
-                <origin rpy="0 0 0" xyz="0.03997881004884705 -0.0005082075189353901 -0.03926307553084657"/>
-                <mass value="2.1436339240369744"/>
-                <inertia ixx="0.008938" ixy="7e-06" ixz="0.000553" iyy="0.009241" iyz="-0.000113" izz="0.000887"/>
+                <origin rpy="0 0 0" xyz="0.04071287283172147 -8.153806755863768e-05 -0.04195721621845735"/>
+                <mass value="2.4245187944339057"/>
+                <inertia ixx="0.00996" ixy="1e-06" ixz="0.000598" iyy="0.01031" iyz="0.000146" izz="0.00104"/>
             </inertial>
             <visual>
                 <origin rpy="0 0 0" xyz="0 0 0"/>
                 <geometry>
-                    <mesh filename="package://storz_exoscope_description/meshes/visual/link_0.stl" scale="0.001 0.001 0.001"/>
+                    <mesh filename="package://storz_straight_exoscope_hsi_description/meshes/visual/link_0.stl" scale="0.001 0.001 0.001"/>
                 </geometry>
                 <material name="silver">
@@ -29,10 +29,10 @@
                 <origin rpy="0 0 0" xyz="0 0 0"/>
                 <geometry>
-                    <mesh filename="package://storz_exoscope_description/meshes/collision/link_0.stl" scale="0.001 0.001 0.001"/>
+                    <mesh filename="package://storz_straight_exoscope_hsi_description/meshes/collision/link_0.stl" scale="0.001 0.001 0.001"/>
                 </geometry>
             </collision>
         </link>
         <joint name="${exoscope_name}_joint_cm" type="fixed">
-            <origin rpy="0 0 -1.57079632679" xyz="0.047 -0.005826 0.115248"/>
+            <origin rpy="-1.57079632679 -1.57079632679 0" xyz="0.046594 0.000596 0.1205"/>
             <parent link="${exoscope_name}_link_0"/>
             <child link="${exoscope_name}_link_cm"/>
@@ -50,5 +50,5 @@
         </link>
         <!-- extensions -->
-        <xacro:storz_exoscope_gazebo exoscope_name="${exoscope_name}" robot_name="${robot_name}"/>
+        <xacro:storz_straight_exoscope_hsi_gazebo exoscope_name="${exoscope_name}" robot_name="${robot_name}"/>
     </xacro:macro>
 </robot>

File: storz_tilt_endoscope_description/urdf/storz_tilt_endoscope_description.urdf.xacro (robot description, xacro)
@@ -3,5 +3,5 @@
     <xacro:macro name="storz_tilt_endoscope" params="tilt_endoscope_name robot_name parent">
         <!-- include gazebo specifications -->
-        <xacro:include filename="$(find storz_tilt_endoscope_description)/urdf/storz_tilt_endoscope.gazebo.xacro" />
+        <xacro:include filename="$(find storz_tilt_endoscope_description)/gazebo/storz_tilt_endoscope.gazebo.xacro" />
         <!--joint between {parent} and link_0-->
         <joint name="${parent}_${tilt_endoscope_name}_joint" type="fixed">

Commit message: corrected colors

File: da_vinci_endoscope_description/urdf/da_vinci_endoscope_description.urdf.xacro (robot description, xacro)
@@ -50,6 +50,6 @@
                     <mesh filename="package://da_vinci_endoscope_description/meshes/visual/link_1.stl"/>
                 </geometry>
-                <material name="silver">
-                    <color rgba="1 0 0 1"/>
+                <material name="white">
+                    <color rgba="1.0 1.0 1.0 1.0"/>
                 </material>
             </visual>

File: storz_endoscope_description/urdf/storz_endoscope_description.urdf.xacro (robot description, xacro)
@@ -22,6 +22,6 @@
                     <mesh filename="package://storz_endoscope_description/meshes/visual/link_0.stl" scale="0.001 0.001 0.001"/>
                 </geometry>
-                <material name="silver">
-                    <color rgba="1 0 0 1"/>
+                <material name="white">
+                    <color rgba="1.0 1.0 1.0 1.0"/>
                 </material>
             </visual>
@@ -50,6 +50,6 @@
                     <mesh filename="package://storz_endoscope_description/meshes/visual/link_1.stl" scale="0.001 0.001 0.001"/>
                 </geometry>
-                <material name="silver">
-                    <color rgba="1 0 0 1"/>
+                <material name="white">
+                    <color rgba="1.0 1.0 1.0 1.0"/>
                 </material>
             </visual>

File: storz_exoscope_description/urdf/storz_exoscope_description.urdf.xacro (robot description, xacro)
@@ -22,6 +22,6 @@
                     <mesh filename="package://storz_exoscope_description/meshes/visual/link_0.stl" scale="0.001 0.001 0.001"/>
                 </geometry>
-                <material name="silver">
-                    <color rgba="1 0 0 1"/>
+                <material name="white">
+                    <color rgba="1.0 1.0 1.0 1.0"/>
                 </material>
             </visual>

File: storz_straight_exoscope_hsi_description/urdf/storz_straight_exoscope_hsi_description.urdf.xacro (robot description, xacro)
@@ -22,6 +22,6 @@
                     <mesh filename="package://storz_straight_exoscope_hsi_description/meshes/visual/link_0.stl" scale="0.001 0.001 0.001"/>
                 </geometry>
-                <material name="silver">
-                    <color rgba="1 0 0 1"/>
+                <material name="white">
+                    <color rgba="1.0 1.0 1.0 1.0"/>
                 </material>
             </visual>

File: storz_tilt_endoscope_description/urdf/storz_tilt_endoscope_description.urdf.xacro (robot description, xacro)
@@ -22,6 +22,6 @@
                     <mesh filename="package://storz_tilt_endoscope_description/meshes/visual/link_0.stl" scale="0.001 0.001 0.001"/>
                 </geometry>
-                <material name="silver">
-                    <color rgba="1 0 0 1"/>
+                <material name="white">
+                    <color rgba="1.0 1.0 1.0 1.0"/>
                 </material>
             </visual>
@@ -50,6 +50,6 @@
                     <mesh filename="package://storz_tilt_endoscope_description/meshes/visual/link_1.stl" scale="0.001 0.001 0.001"/>
                 </geometry>
-                <material name="silver">
-                    <color rgba="1 0 0 1"/>
+                <material name="white">
+                    <color rgba="1.0 1.0 1.0 1.0"/>
                 </material>
             </visual>
