Commit message: updated rotations

File: storz_exoscope_description/urdf/storz_exoscope.xacro (robot description, xacro)
@@ -8,5 +8,5 @@
             <parent link="${parent}"/>
             <child link="${exoscope_name}_link_0"/>
-            <origin xyz="0 0 0" rpy="0 0 1.57079632679"/>
+            <origin xyz="0 0 0" rpy="0 -1.57079632679 1.57079632679"/>
         </joint>
         <!-- link 0 -->
@@ -34,5 +34,5 @@
         </link>
         <joint name="${exoscope_name}_joint_cm" type="fixed">
-            <origin rpy="0 0 0" xyz="0.047 -0.005826 0.115248"/>
+            <origin rpy="0 0 -1.57079632679" xyz="0.047 -0.005826 0.115248"/>
             <parent link="${exoscope_name}_link_0"/>
             <child link="${exoscope_name}_link_cm"/>
