Commit message: corrected camera orientation

File: storz_tilt_endoscope_description/urdf/storz_tilt_endoscope.xacro (robot description, xacro)
@@ -62,5 +62,5 @@
         </link>
         <joint name="${tilt_endoscope_name}_joint_cm" type="fixed">
-            <origin rpy="0 0 0" xyz="0.0 0.0 0.2874"/>
+            <origin rpy="-1.57079632679 -1.57079632679 0" xyz="0.0 0.0 0.2874"/>
             <parent link="${tilt_endoscope_name}_link_1"/>
             <child link="${tilt_endoscope_name}_link_cm"/>
