Commit message: configured camera orientation

File: storz_straight_exoscope_hsi_description/urdf/storz_straight_exoscope_hsi.xacro (robot description, xacro)
@@ -34,5 +34,5 @@
         </link>
         <joint name="${exoscope_name}_joint_cm" type="fixed">
-            <origin rpy="0 0 0" xyz="0.046594 0.000596 0.1205"/>
+            <origin rpy="-1.57079632679 -1.57079632679 0" xyz="0.046594 0.000596 0.1205"/>
             <parent link="${exoscope_name}_link_0"/>
             <child link="${exoscope_name}_link_cm"/>
